File: Thermal-Mint-HW/TM-Power.kicad_sch (KiCad schematic)
At the start: 0 parts

Commit message: Clean up of output circuits
Parts:
- added C28, C29, C30, C31: 470n, Capacitor_SMD:C_0603_1608Metric_Pad1.08x0.95mm_HandSolder, symbol Device:C
- added U5: NCP1117-3.3_SOT223, Package_TO_SOT_SMD:SOT-223-3_TabPin2, symbol Regulator_Linear:NCP1117-3.3_SOT223
Connections:
- new net +3V3: C30.1, C31.1, U5.2 (VO)
- new net +5V: C28.1, C29.1, U5.3 (VI)
- new net GND: C28.2, C29.2, C30.2, C31.2, U5.1 (GND)
Changed lines of the file:
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@@
-(kicad_sch (version 20210621) (generator eeschema)
+(kicad_sch (version 20211123) (generator eeschema)
   (paper "A4")
+  (junction (at 143.51 118.11) (diameter 0) (color 0 0 0 0)
+  )
+  (junction (at 113.665 118.11) (diameter 0) (color 0 0 0 0)
+  )
+  (junction (at 97.79 118.11) (diameter 0) (color 0 0 0 0)
+  )
+  (junction (at 153.67 118.11) (diameter 0) (color 0 0 0 0)
+  )
+  (junction (at 107.95 118.11) (diameter 0) (color 0 0 0 0)
+  )
+  (wire (pts (xy 143.51 118.11) (xy 134.62 118.11))
+    (stroke (width 0) (type default) (color 0 0 0 0))
+  )
+  (wire (pts (xy 107.95 118.11) (xy 97.79 118.11))
+    (stroke (width 0) (type default) (color 0 0 0 0))
+  )
+  (wire (pts (xy 113.665 118.11) (xy 107.95 118.11))
+    (stroke (width 0) (type default) (color 0 0 0 0))
+  )
+  (wire (pts (xy 119.38 118.11) (xy 113.665 118.11))
+    (stroke (width 0) (type default) (color 0 0 0 0))
+  )
+  (wire (pts (xy 153.67 118.11) (xy 143.51 118.11))
+    (stroke (width 0) (type default) (color 0 0 0 0))
+  )
+  (wire (pts (xy 153.67 118.11) (xy 165.1 118.11))
+    (stroke (width 0) (type default) (color 0 0 0 0))
+  )
+  (wire (pts (xy 97.79 118.11) (xy 88.9 118.11))
+    (stroke (width 0) (type default) (color 0 0 0 0))
+  )
+  (hierarchical_label "Vin" (shape input) (at 88.9 118.11 180)
+    (effects (font (size 1.27 1.27)) (justify right))
+  )
+  (symbol (lib_id "Device:C") (at 153.67 121.92 0) (unit 1)
+    (in_bom yes) (on_board yes)
+    (property "Reference" "C31" (id 0) (at 154.305 119.38 0)
+      (effects (font (size 1.27 1.27)) (justify left))
+    )
+    (property "Value" "470n" (id 1) (at 154.305 124.46 0)
+      (effects (font (size 1.27 1.27)) (justify left))
+    )
+    (property "Footprint" "Capacitor_SMD:C_0603_1608Metric_Pad1.08x0.95mm_HandSolder" (id 2) (at 154.6352 125.73 0)
+      (effects (font (size 1.27 1.27)) hide)
+    )
+    (property "Datasheet" "~" (id 3) (at 153.67 121.92 0)
+      (effects (font (size 1.27 1.27)) hide)
+    )
+    (pin "1")
+    (pin "2")
+  )
+  (symbol (lib_id "power:GND") (at 107.95 125.73 0) (unit 1)
+    (in_bom yes) (on_board yes)
+    (property "Reference" "#PWR045" (id 0) (at 107.95 132.08 0)
+      (effects (font (size 1.27 1.27)) hide)
+    )
+    (property "Value" "GND" (id 1) (at 107.95 129.54 0))
+    (property "Footprint" "" (id 2) (at 107.95 125.73 0)
+      (effects (font (size 1.27 1.27)) hide)
+    )
+    (property "Datasheet" "" (id 3) (at 107.95 125.73 0)
+      (effects (font (size 1.27 1.27)) hide)
+    )
+    (pin "1")
+  )
+  (symbol (lib_id "power:GND") (at 97.79 125.73 0) (unit 1)
+    (in_bom yes) (on_board yes)
+    (property "Reference" "#PWR044" (id 0) (at 97.79 132.08 0)
+      (effects (font (size 1.27 1.27)) hide)
+    )
+    (property "Value" "GND" (id 1) (at 97.79 129.54 0))
+    (property "Footprint" "" (id 2) (at 97.79 125.73 0)
+      (effects (font (size 1.27 1.27)) hide)
+    )
+    (property "Datasheet" "" (id 3) (at 97.79 125.73 0)
+      (effects (font (size 1.27 1.27)) hide)
+    )
+    (pin "1")
+  )
+  (symbol (lib_id "power:GND") (at 153.67 125.73 0) (unit 1)
+    (in_bom yes) (on_board yes)
+    (property "Reference" "#PWR048" (id 0) (at 153.67 132.08 0)
+      (effects (font (size 1.27 1.27)) hide)
+    )
+    (property "Value" "GND" (id 1) (at 153.67 129.54 0))
+    (property "Footprint" "" (id 2) (at 153.67 125.73 0)
+      (effects (font (size 1.27 1.27)) hide)
+    )
+    (property "Datasheet" "" (id 3) (at 153.67 125.73 0)
+      (effects (font (size 1.27 1.27)) hide)
+    )
+    (pin "1")
+  )
+  (symbol (lib_id "power:GND") (at 143.51 125.73 0) (unit 1)
+    (in_bom yes) (on_board yes)
+    (property "Reference" "#PWR047" (id 0) (at 143.51 132.08 0)
+      (effects (font (size 1.27 1.27)) hide)
+    )
+    (property "Value" "GND" (id 1) (at 143.51 129.54 0))
+    (property "Footprint" "" (id 2) (at 143.51 125.73 0)
+      (effects (font (size 1.27 1.27)) hide)
+    )
+    (property "Datasheet" "" (id 3) (at 143.51 125.73 0)
+      (effects (font (size 1.27 1.27)) hide)
+    )
+    (pin "1")
+  )
+  (symbol (lib_id "Device:C") (at 107.95 121.92 0) (unit 1)
+    (in_bom yes) (on_board yes)
+    (property "Reference" "C29" (id 0) (at 108.585 119.38 0)
+      (effects (font (size 1.27 1.27)) (justify left))
+    )
+    (property "Value" "470n" (id 1) (at 108.585 124.46 0)
+      (effects (font (size 1.27 1.27)) (justify left))
+    )
+    (property "Footprint" "Capacitor_SMD:C_0603_1608Metric_Pad1.08x0.95mm_HandSolder" (id 2) (at 108.9152 125.73 0)
+      (effects (font (size 1.27 1.27)) hide)
+    )
+    (property "Datasheet" "~" (id 3) (at 107.95 121.92 0)
+      (effects (font (size 1.27 1.27)) hide)
+    )
+    (pin "1")
+    (pin "2")
+  )
+  (symbol (lib_id "Device:C") (at 143.51 121.92 0) (unit 1)
+    (in_bom yes) (on_board yes)
+    (property "Reference" "C30" (id 0) (at 144.145 119.38 0)
+      (effects (font (size 1.27 1.27)) (justify left))
+    )
+    (property "Value" "470n" (id 1) (at 144.145 124.46 0)
+      (effects (font (size 1.27 1.27)) (justify left))
+    )
+    (property "Footprint" "Capacitor_SMD:C_0603_1608Metric_Pad1.08x0.95mm_HandSolder" (id 2) (at 144.4752 125.73 0)
+      (effects (font (size 1.27 1.27)) hide)
+    )
+    (property "Datasheet" "~" (id 3) (at 143.51 121.92 0)
+      (effects (font (size 1.27 1.27)) hide)
+    )
+    (pin "1")
+    (pin "2")
+  )
+  (symbol (lib_id "Regulator_Linear:NCP1117-3.3_SOT223") (at 127 118.11 0) (unit 1)
+    (in_bom yes) (on_board yes) (fields_autoplaced)
+    (property "Reference" "U5" (id 0) (at 127 112.5052 0))
+    (property "Value" "NCP1117-3.3_SOT223" (id 1) (at 127 115.0421 0))
+    (property "Footprint" "Package_TO_SOT_SMD:SOT-223-3_TabPin2" (id 2) (at 127 113.03 0)
+      (effects (font (size 1.27 1.27)) hide)
+    )
+    (property "Datasheet" "http://www.onsemi.com/pub_link/Collateral/NCP1117-D.PDF" (id 3) (at 129.54 124.46 0)
+      (effects (font (size 1.27 1.27)) hide)
+    )
+    (pin "1")
+    (pin "2")
+    (pin "3")
+  )
+  (symbol (lib_id "Device:C") (at 97.79 121.92 0) (unit 1)
+    (in_bom yes) (on_board yes)
+    (property "Reference" "C28" (id 0) (at 98.425 119.38 0)
+      (effects (font (size 1.27 1.27)) (justify left))
+    )
+    (property "Value" "470n" (id 1) (at 98.425 124.46 0)
+      (effects (font (size 1.27 1.27)) (justify left))
+    )
+    (property "Footprint" "Capacitor_SMD:C_0603_1608Metric_Pad1.08x0.95mm_HandSolder" (id 2) (at 98.7552 125.73 0)
+      (effects (font (size 1.27 1.27)) hide)
+    )
+    (property "Datasheet" "~" (id 3) (at 97.79 121.92 0)
+      (effects (font (size 1.27 1.27)) hide)
+    )
+    (pin "1")
+    (pin "2")
+  )
+  (symbol (lib_id "power:+5V") (at 113.665 118.11 0) (unit 1)
+    (in_bom yes) (on_board yes) (fields_autoplaced)
+    (property "Reference" "#PWR063" (id 0) (at 113.665 121.92 0)
+      (effects (font (size 1.27 1.27)) hide)
+    )
+    (property "Value" "+5V" (id 1) (at 113.665 114.5342 0))
+    (property "Footprint" "" (id 2) (at 113.665 118.11 0)
+      (effects (font (size 1.27 1.27)) hide)
+    )
+    (property "Datasheet" "" (id 3) (at 113.665 118.11 0)
+      (effects (font (size 1.27 1.27)) hide)
+    )
+    (pin "1")
+  )
+  (symbol (lib_id "power:GND") (at 127 125.73 0) (unit 1)
+    (in_bom yes) (on_board yes)
+    (property "Reference" "#PWR046" (id 0) (at 127 132.08 0)
+      (effects (font (size 1.27 1.27)) hide)
+    )
+    (property "Value" "GND" (id 1) (at 127 129.54 0))
+    (property "Footprint" "" (id 2) (at 127 125.73 0)
+      (effects (font (size 1.27 1.27)) hide)
+    )
+    (property "Datasheet" "" (id 3) (at 127 125.73 0)
+      (effects (font (size 1.27 1.27)) hide)
+    )
+    (pin "1")
+  )
+  (symbol (lib_id "power:+3V3") (at 165.1 118.11 0) (unit 1)
+    (in_bom yes) (on_board yes) (fields_autoplaced)
+    (property "Reference" "#PWR049" (id 0) (at 165.1 121.92 0)
+      (effects (font (size 1.27 1.27)) hide)
+    )
+    (property "Value" "+3V3" (id 1) (at 165.1 113.03 0))
+    (property "Footprint" "" (id 2) (at 165.1 118.11 0)
+      (effects (font (size 1.27 1.27)) hide)
+    )
+    (property "Datasheet" "" (id 3) (at 165.1 118.11 0)
+      (effects (font (size 1.27 1.27)) hide)
+    )
+    (pin "1")
+  )
 )
